Commit message: bringup - real hardware

File: omo_r1_description/urdf/omo_r1.gazebo.xacro (robot description, xacro)
@@ -78,5 +78,5 @@
       <leftJoint>wheel_left_joint</leftJoint>
       <rightJoint>wheel_right_joint</rightJoint>
-      <wheelSeparation>0.590</wheelSeparation>
+      <wheelSeparation>0.591</wheelSeparation>
       <wheelDiameter>0.220</wheelDiameter>
       <wheelAcceleration>1</wheelAcceleration>

File: omo_r1_description/urdf/omo_r1.urdf.xacro (robot description, xacro)
@@ -150,5 +150,5 @@
     <parent link="base_link"/>
     <child link="imu_link"/>
-    <origin xyz="0.0 0 0.190" rpy="0 0 0"/>
+    <origin xyz="0.0 0 0.190" rpy="0 0 1.5758"/>
   </joint>
   <link name="imu_link"/>
