Commit message: modified for package redefinition

File: omo_r1_description/urdf/common_properties.xacro (robot description, xacro)
@@ -1,5 +1,5 @@
 <?xml version="1.0" ?>
 <robot name="xacro_properties" xmlns:xacro="http://ros.org/wiki/xacro">
-  <!-- Init colour -->
+  <!-- Init color -->
   <material name="black">
       <color rgba="0.0 0.0 0.0 1.0"/>

File: omo_r1_description/urdf/omo_r1.urdf.xacro (robot description, xacro)
@@ -2,5 +2,4 @@
 <robot name="omo_r1" xmlns:xacro="http://ros.org/wiki/xacro">
   <xacro:include filename="$(find omo_r1_description)/urdf/common_properties.xacro"/>
-  <xacro:include filename="$(find omo_r1_description)/urdf/omo_r1.gazebo.xacro"/>
   <link name="base_footprint"/>
   <joint name="base_joint" type="fixed">
@@ -13,5 +12,5 @@
       <origin xyz="0.097 0.276 0.19" rpy="3.14 0 -1.57"/>
       <geometry>
-        <mesh filename="package://omo_r1_description/meshes/bases/R1_body.stl" scale="0.001 0.001 0.001"/>
+        <mesh filename="package://omo_r1_description/meshes/bases/omo_r1_body.stl" scale="0.001 0.001 0.001"/>
       </geometry>
       <material name="light_black"/>
@@ -20,5 +19,5 @@
       <origin xyz="0.097 0.276 0.19" rpy="3.14 0 -1.57"/>
       <geometry>
-        <mesh filename="package://omo_r1_description/meshes/bases/R1_body.stl" scale="0.001 0.001 0.001"/>
+        <mesh filename="package://omo_r1_description/meshes/bases/omo_r1_body.stl" scale="0.001 0.001 0.001"/>
       </geometry>
     </collision>
@@ -41,5 +40,5 @@
       <origin xyz="-0.1105 -0.06 0.1104" rpy="-1.57 0 0"/>
       <geometry>
-        <mesh filename="package://omo_r1_description/meshes/wheels/wheel.stl" scale="0.001 0.001 0.001"/>
+        <mesh filename="package://omo_r1_description/meshes/wheels/omo_r1_wheel.stl" scale="0.001 0.001 0.001"/>
       </geometry>
       <material name="dark"/>
@@ -48,5 +47,5 @@
       <origin xyz="-0.1105 -0.06 0.1104" rpy="-1.57 0 0"/>
       <geometry>
-        <mesh filename="package://omo_r1_description/meshes/wheels/wheel.stl" scale="0.001 0.001 0.001"/>
+        <mesh filename="package://omo_r1_description/meshes/wheels/omo_r1_wheel.stl" scale="0.001 0.001 0.001"/>
       </geometry>
     </collision>
@@ -69,5 +68,5 @@
       <origin xyz="-0.110 0.06 -0.1103" rpy="1.57 0 0"/>
       <geometry>
-        <mesh filename="package://omo_r1_description/meshes/wheels/wheel.stl" scale="0.001 0.001 0.001"/>
+        <mesh filename="package://omo_r1_description/meshes/wheels/omo_r1_wheel.stl" scale="0.001 0.001 0.001"/>
       </geometry>
       <material name="dark"/>
@@ -76,5 +75,5 @@
       <origin xyz="-0.110 0.06 -0.1103" rpy="1.57 0 0"/>
       <geometry>
-        <mesh filename="package://omo_r1_description/meshes/wheels/wheel.stl" scale="0.001 0.001 0.001"/>
+        <mesh filename="package://omo_r1_description/meshes/wheels/omo_r1_wheel.stl" scale="0.001 0.001 0.001"/>
       </geometry>
     </collision>
@@ -87,24 +86,4 @@
       </inertial>
   </link>
-  <!-- <joint name="caster_back_joint" type="fixed">
-    <parent link="base_link"/>
-    <child link="caster_back_link"/>
-    <origin xyz="-0.33 0.0 0.06" rpy="0 0 0"/>
-  </joint>
-  <link name="caster_back_link">
-    <collision>
-      <origin xyz="0 0.000 -0.133" rpy="0 0 0"/>
-      <geometry>
-        <box size="0.01 0.01 0.01"/>
-      </geometry>
-    </collision>
-    <inertial>
-      <origin xyz="0 0 0" />
-      <mass value="0.005" />
-      <inertia ixx="0.001" ixy="0.0" ixz="0.0"
-               iyy="0.001" iyz="0.0"
-               izz="0.001" />
-    </inertial>
-  </link> -->
   <joint name="caster_back_right_joint" type="fixed">
     <parent link="base_link"/>
@@ -162,5 +141,5 @@
       <origin xyz="0 0 0.0" rpy="0.0 0 0.0"/>
       <geometry>
-        <mesh filename="package://omo_r1_description/meshes/sensors/lds.stl" scale="0.001 0.001 0.001"/>
+        <mesh filename="package://omo_r1_description/meshes/sensors/omo_r1_lidar.stl" scale="0.001 0.001 0.001"/>
       </geometry>
       <material name="dark"/>
@@ -169,5 +148,5 @@
       <origin xyz="0 0 0.0" rpy="0.0 0 0.0"/>
       <geometry>
-        <mesh filename="package://omo_r1_description/meshes/sensors/lds.stl" scale="0.001 0.001 0.001"/>
+        <mesh filename="package://omo_r1_description/meshes/sensors/omo_r1_lidar.stl" scale="0.001 0.001 0.001"/>
       </geometry>
     </collision>
@@ -180,18 +159,3 @@
     </inertial>
   </link>
-<!--
-  <joint name="camera_joint" type="fixed">
-    <origin xyz="0.073 -0.011 0.084" rpy="0 0 0"/>
-    <parent link="base_link"/>
-    <child link="camera_link"/>
-  </joint>
-  <link name="camera_link">
-    <collision>
-      <origin xyz="0.005 0.011 0.013" rpy="0 0 0"/>
-      <geometry>
-        <box size="0.015 0.030 0.027"/>
-      </geometry>
-    </collision>
-  </link>
--->
 </robot>
