Commit message: lidar mount modification as h/w wise

File: omo_r1_description/urdf/omo_r1.urdf.xacro (robot description, xacro)
@@ -135,5 +135,5 @@
     <parent link="base_link"/>
     <child link="base_scan"/>
-    <origin xyz="0.10 0 0.230" rpy="0.0 0 0.0"/>
+    <origin xyz="0.06 0 0.230" rpy="0.0 0 3.14159"/>
   </joint>
   <link name="base_scan">

Commit message: image recognition - ar marker tracking package added

File: omo_r1_description/urdf/omo_r1.urdf.xacro (robot description, xacro)
@@ -159,3 +159,35 @@
     </inertial>
   </link>
+  <joint name="camera_joint" type="fixed">
+    <origin xyz="0.07 0.0 0.35" rpy="0 0 0"/>
+    <parent link="base_link"/>
+    <child link="camera_link"/>
+  </joint>
+  <link name="camera_link">
+    <visual>
+      <origin xyz="0 0 0.0" rpy="1.5758 0.0 1.5758"/>
+      <geometry>
+        <mesh filename="package://omo_r1_description/meshes/sensors/omo_r1_camera.stl" scale="0.001 0.001 0.001"/>
+      </geometry>
+      <material name="dark"/>
+    </visual>
+    <collision>
+      <origin xyz="0 0 0.0" rpy="1.5758 0.0 1.5758"/>
+      <geometry>
+        <mesh filename="package://omo_r1_description/meshes/sensors/omo_r1_camera.stl" scale="0.001 0.001 0.001"/>
+      </geometry>
+    </collision>
+  </link>
+  <joint name="camera_rgb_joint" type="fixed">
+    <origin xyz="0.03 0.0 0.0" rpy="0 0 0"/>
+    <parent link="camera_link"/>
+    <child link="camera_rgb_frame"/>
+  </joint>
+  <link name="camera_rgb_frame"/>
+  <joint name="camera_rgb_optical_joint" type="fixed">
+    <origin xyz="0 0 0" rpy="-1.57 0 -1.57"/>
+    <parent link="camera_rgb_frame"/>
+    <child link="camera_rgb_optical_frame"/>
+  </joint>
+  <link name="camera_rgb_optical_frame"/>
 </robot>

Commit message: marker_slam

File: omo_r1_description/urdf/omo_r1.urdf.xacro (robot description, xacro)
@@ -160,5 +160,5 @@
   </link>
   <joint name="camera_joint" type="fixed">
-    <origin xyz="0.07 0.0 0.35" rpy="0 0 0"/>
+    <origin xyz="0.07 0.0 0.63" rpy="0 0.7 0"/>
     <parent link="base_link"/>
     <child link="camera_link"/>
